File: FluxDrive.kicad_sch (KiCad schematic)
At the start: 119 parts, among them J1 Amiga floppy 34, J2 Floppy power, J3 USB-C, J4 UART / recovery, J5 Spare GPIO, SW1 BOOT, SW2 RESET, U1 ESP32-S3-WROOM-1-N16R8, U2 74LVC14A, U3 74LVC14A, U4 74LVC07A, U5 TPS259531, U6 TLV62569DBVR, U7 USBLC6-2SC6

Commit message: Schematic review: fix VBUS back-feed and stale-netlist tests, take in the minors
Four reviews of the generated schematic (bus, power, ESP32-S3, PCB and code),
recorded in docs/reviews/2026-09-29-schematic-review.md.

- U7 (USBLC6) supply pin on +3V3 instead of VBUS, 10k bleeder on VBUS (SPWR-1)
- tests read a netlist exported fresh from the committed schematic and fail
  when it is not what hardware/design.py generates (SCODE-1)
- AMIGA_PWR divider 1k/1k5: low on USB alone (SESP-1, SPWR-4)
- +5V_A bulk 2 x 47uF 10V instead of 100uF 6.3V (SPCB-2)
- J2 vertical TE 171825-4 (C210162) with its own footprint (SPCB-1)
- unfitted pads: V5SYS damper, SMAJ13A on +5V_IN, 15pF feed-forward, all 0603
- generator: pin assigned twice and stacked pins on different nets raise,
  unit in the pin/label IDs, in_pos_files only for fitted BOM parts
- tests: gate pairing, unfitted pads, USB-alone DC levels, full-severity ERC
- spec v0.3 with the review's corrections
Parts:
- added C21, C22: 10pF, Capacitor_SMD:C_0603_1608Metric, symbol Device:C
- added D4: SMAJ13A, Diode_SMD:D_SMA, symbol Diode:SMAJ13A
- added R61: 470, Resistor_SMD:R_0402_1005Metric, symbol Device:R
- added R62: 1K, Resistor_SMD:R_0402_1005Metric, symbol Device:R
- C1, C2, C3, C4: footprint Capacitor_SMD:C_0402_1005Metric -> Capacitor_SMD:C_0603_1608Metric
- C10: value 100uF -> 47uF; LCSC C15008 -> C96123
- C11: value 100nF -> 47uF; footprint Capacitor_SMD:C_0402_1005Metric -> Capacitor_SMD:C_1206_3216Metric; LCSC C1525 -> C96123
- C12: value 10uF -> 100nF; footprint Capacitor_SMD:C_0603_1608Metric -> Capacitor_SMD:C_0402_1005Metric; LCSC C19702 -> C1525
- C13: value 100nF -> 10uF; footprint Capacitor_SMD:C_0402_1005Metric -> Capacitor_SMD:C_0603_1608Metric; LCSC C1525 -> C19702
- C14: value 6.8pF -> 100nF; LCSC (none) -> C1525; now fitted; now in the parts list
- C15: value 22uF -> 4.7uF; footprint Capacitor_SMD:C_0805_2012Metric -> Capacitor_SMD:C_0603_1608Metric; LCSC C45783 -> (none); now not fitted; now left out of the parts list
- C16: value 22uF -> 15pF; footprint Capacitor_SMD:C_0805_2012Metric -> Capacitor_SMD:C_0603_1608Metric; LCSC C45783 -> (none); now not fitted; now left out of the parts list
- C17: value 100nF -> 22uF; footprint Capacitor_SMD:C_0402_1005Metric -> Capacitor_SMD:C_0805_2012Metric; LCSC C1525 -> C45783
- C18: value 1uF -> 22uF; footprint Capacitor_SMD:C_0402_1005Metric -> Capacitor_SMD:C_0805_2012Metric; LCSC C52923 -> C45783
- C19: value 10pF -> 100nF; LCSC (none) -> C1525; now fitted; now in the parts list
- C20: value 10pF -> 1uF; LCSC (none) -> C52923; now fitted; now in the parts list
- J2: footprint FluxDrive:171826-4 -> FluxDrive:171825-4; symbol FluxDrive:171826-4 -> FluxDrive:171825-4; LCSC C590635 -> C210162
- R16, R25: footprint Resistor_SMD:R_0402_1005Metric -> Resistor_SMD:R_0603_1608Metric
- R49: value 100K -> 1R; footprint Resistor_SMD:R_0402_1005Metric -> Resistor_SMD:R_0603_1608Metric; LCSC C25741 -> (none); now not fitted; now left out of the parts list
- R50: value 22K -> 100K; LCSC C25768 -> C25741
- R51: value 10K -> 22K; LCSC C25744 -> C25768
- R52: value 15K -> 1K; LCSC C25756 -> C11702
- R53: value 10K -> 1K5; LCSC C25744 -> C25867
- R55: value 5K1 -> 10K; LCSC C25905 -> C25744
- R57: value 22 -> 5K1; LCSC C25092 -> C25905
- R58: value 22 -> 10K; LCSC C25092 -> C25744
- R59: value 470 -> 22; LCSC C25117 -> C25092
- R60: value 1K -> 22; LCSC C11702 -> C25092
Connections:
- net +3V3: now also C18.1, C19.1, R50.1, R55.1, U7.5 (VBUS); no longer C14.1, C15.1, R49.1, R53.1
- net +5V_A: now also C12.1, R52.1; no longer R51.1
- net +5V_IN: now also D4.1 (A1)
- net AMIGA_PWR: now also R52.2, R53.1; no longer R51.2, R52.1
- net BOOT: now also R55.2; no longer R54.2
- net BUCK_FB: now also C16.2, R50.2, R51.1; no longer C14.2, R49.2, R50.1
- net ESP_EN: now also C20.1, R54.2; no longer C18.1, R53.2
- net ESP_TXD0: now also R61.1; no longer R59.1
- net GND: now also C14.2, R51.2, R53.2, R57.2, R58.2, C21.2, C22.2, D4.2 (A2); no longer C16.2, R50.2, R52.2, R55.2
- net LED: now also R62.1; no longer R60.1
- net LED_A: now also R62.2; no longer R60.2
- net UART_TX: now also R61.2; no longer R59.2
- net USB_CC1: now also R56.1; no longer R55.1
- net USB_CC2: now also R57.1; no longer R56.1
- net USB_DN: now also R60.2, C22.1; no longer C20.1, R58.2
- net USB_DN_C: now also R60.1; no longer R58.1
- net USB_DP: now also R59.2, C21.1; no longer C19.1, R57.2
- net USB_DP_C: now also R59.1; no longer R57.1
- net V5SYS: now also C14.1, R49.1; no longer C12.1
- net VBUS: now also R58.1; no longer U7.5 (VBUS)
- new net V5SYS_DAMP: C15.1, R49.2
Other:
- moved on the sheet: C10, C11, C12, C13, C17, C18, C8, C9, D1, D2, L1, R46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

Commit message: Board: footprints from the netlist, outline and placement
- tools/pcb_sync.py (from the Nano-Tek tool, without its Rev 1.2 migration) builds
  FluxDrive.kicad_pcb from the netlist; tools/pcb_place.py sets the 60 x 48 mm outline,
  the GND pours and every position, moving non-fixed parts to the nearest free spot
- module footprint copy with 0.3 mm thermal vias; netclass patterns with the / prefix,
  Power tracks 0.3 mm (the eFuse pads are 0.25 mm at 0.5 mm pitch)
- tests/test_pcb.py: outline, J1 on the south edge, antenna past the north edge,
  J2 beside J1
Parts:
- U1: footprint RF_Module:ESP32-S3-WROOM-1 -> FluxDrive:ESP32-S3-WROOM-1
Changed lines of the file:
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@@
 			)
 		)
-		(property "Footprint" "RF_Module:ESP32-S3-WROOM-1"
+		(property "Footprint" "FluxDrive:ESP32-S3-WROOM-1"
 			(at 48.26 367.03 0)
 			(hide yes)

Commit message: Layout review and fixes: 4 layers, antenna on the board
Four specialist reviews of the task-10 layout (55 findings, 13 major); the
record with every decision is docs/reviews/2026-09-29-layout-review.md.

- 4 layers (Dimitri): In1 solid GND, In2 solid +3V3; every GND/+3V3 pad
  has its own via, outer pours stitched to In1.
- The board grows 6.5 mm north; the module's antenna lies 0.5 mm inside
  the edge over copper-free board (Dimitri; O10 closed). Spec v0.4.
- Buffer gates re-assigned in connector order (U3 pins 4-16, U2 18-32);
  row B follows the buffer inputs; schematic and PDF regenerated.
- Rule areas: J1 rows, antenna edge, buck, module underside, USB-C body.
- Hand routes before Freerouting: VBUS bridge, +5V_A rail, eFuse, USB
  D+/D- pad joins, /DKRD_D (6.4 mm, no via).
- Build scripts: deterministic fan-out, planes in the DSN, varied
  Freerouting runs, pads' own clearance in the stitching, placement check,
  fit template with scale bars, note and STEP.

Build 12: DRC 0 errors, 0 unconnected, 0 parity; 71 tests pass.
Connections:
- net DIR: now also U2.2; no longer U2.4
- net DIR_B: now also U2.1; no longer U2.3
- net DKRD_D: now also U4.4; no longer U4.2
- net DKRD_N: now also U4.3; no longer U4.1
- net DKWD: now also U2.4; no longer U3.2
- net DKWD_B: now also U2.3; no longer U3.1
- net DKWE: now also U2.10; no longer U3.4
- net DKWE_B: now also U2.11; no longer U3.3
- net GND: now also U2.9; no longer U3.13
- net INDEX_D: now also U4.8; no longer U4.4
- net INDEX_N: now also U4.9; no longer U4.3
- net MTR0: now also U3.8; no longer U2.12
- net MTR0_B: now also U3.9; no longer U2.13
- net MTR0_P4: now also U3.2; no longer U3.6
- net MTR0_P4_B: now also U3.1; no longer U3.5
- net PIN14: now also U3.6; no longer U3.10
- net PIN14_B: now also U3.5; no longer U3.11
- net PIN6: now also U3.12; no longer U3.8
- net PIN6_B: now also U3.13; no longer U3.9
- net RDY_D: now also U4.6; no longer U4.12
- net RDY_N: now also U4.5; no longer U4.13
- net SEL0: now also U3.4; no longer U2.8
- net SEL0_B: now also U3.3; no longer U2.9
- net SEL1: now also U3.10; no longer U2.10
- net SEL1_B: now also U3.11; no longer U2.11
- net STEP: now also U2.12; no longer U2.2
- net STEP_B: now also U2.13; no longer U2.1
- net TRK0_D: now also U4.12; no longer U4.6
- net TRK0_N: now also U4.13; no longer U4.5
- net WPROT_D: now also U4.2; no longer U4.8
- net WPROT_N: now also U4.1; no longer U4.9
Other:
- moved on the sheet: C5, U2B, U2D, U2E, U2F, U2G, U3A, U3B, U3C, U3D, U3E, U3F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

Commit message: Rev B inputs: 4k7 and 1k pull-ups, 1 kOhm to the GPIOs, U3/U2 gates reused
Parts:
- R1, R4, R7: value 1K -> 4K7; LCSC C11702 -> C25900
- R13: value 10K -> 1K; LCSC C25744 -> C11702
- R14, R17: value 100 -> 1K; LCSC C25076 -> C11702
- R15: value 100K -> 100; LCSC C25741 -> C25076
- R16: value 1K -> 100K; footprint Resistor_SMD:R_0603_1608Metric -> Resistor_SMD:R_0402_1005Metric; LCSC (none) -> C25741; now fitted; now in the parts list
- R18: value 100K -> 1K; footprint Resistor_SMD:R_0402_1005Metric -> Resistor_SMD:R_0603_1608Metric; LCSC C25741 -> (none); now not fitted; now left out of the parts list
- R19: value 4K7 -> 100; LCSC C25900 -> C25076
- R20, R29, R32: value 100 -> 100K; LCSC C25076 -> C25741
- R21: value 100K -> 1K; LCSC C25741 -> C11702
- R25: value 1K -> 4K7; footprint Resistor_SMD:R_0603_1608Metric -> Resistor_SMD:R_0402_1005Metric; LCSC (none) -> C25900; now fitted; now in the parts list
- R28: value 10K -> 100; LCSC C25744 -> C25076
- R30: value 100K -> 4K7; footprint Resistor_SMD:R_0402_1005Metric -> Resistor_SMD:R_0603_1608Metric; LCSC C25741 -> (none); now not fitted; now left out of the parts list
- R31: value 10K -> 100; footprint Resistor_SMD:R_0402_1005Metric -> Resistor_SMD:R_0603_1608Metric; LCSC C25744 -> (none); now not fitted; now left out of the parts list
Connections:
- net +3V3: now also R16.2, R20.2, R29.2, R32.2; no longer R15.2, R18.2, R21.2, R28.2, R30.2, R31.2, R33.2
- net +5V_A: now also R14.2, R18.2, R30.2; no longer R13.2, R16.2, R19.2
- net DKWD_B: now also R23.2, R24.1; no longer R20.2, R21.1
- net DKWE_B: now also R26.2, R27.1; no longer R23.2, R24.1
- net GND: now also R33.2; no longer U2.9
- net MTR0: now also R21.1; no longer U1.19 (IO11)
- net MTR0_B: now also R19.2, R20.1; no longer R17.2, R18.1
- net SEL0: now also R13.1; no longer U1.10 (IO17)
- net SEL1: now also R17.1; no longer U1.17 (IO9)
- net SEL1_B: now also R15.2, R16.1; no longer R14.2, R15.1
- net _DKWD: now also R22.1, R23.1; no longer R19.1, R20.1
- net _DKWE: now also R25.1, R26.1; no longer R22.1, R23.1
- net _MTR0: now also R18.1, R19.1; no longer R16.1, R17.1
- net _SEL1: now also R15.1; no longer R13.1
- net SEL_FD_N: now reaches U2.8
- removed net FD_PIN14: J1.14 (Pin_14), R31.1, R32.1
- removed net FD_PIN6: J1.6 (Pin_6), R28.1, R29.1
- net MTR0_P4: no longer names the net of U1.4 (IO4)
- net MTR0_P4: no longer U3.2
- removed net MTR0_P4_B: R26.2, R27.1, U3.1
- net PIN14: no longer names the net of U1.18 (IO10)
- net PIN14: no longer U3.6
- removed net PIN14_B: R32.2, R33.1, U3.5
- net PIN6: no longer names the net of U1.12 (IO8)
- net PIN6: no longer U3.12
- removed net PIN6_B: R29.2, R30.1, U3.13
- removed net _MTR0_P4: J1.4 (Pin_4), R25.1, R26.1
- new net KBRESET: R28.1
- new net M4_MOTOR: U3.6
- new net M4_MTR_N: U3.12
- new net M4_MTR_Q: R33.1, U3.13
- new net MTR0_IO: R21.2, U1.19 (IO11)
- new net MTRX: R30.1, R31.1
- new net MTRX_B: R31.2, R32.1, U3.5
- new net RST_ACT: U3.2
- new net RST_B: R28.2, R29.1, U3.1
- new net SEL0_IO: R13.2, U1.10 (IO17)
- new net SEL1_IO: R17.2, U1.17 (IO9)
- new net SEL_FD: U2.9
- no-connect marks 14 -> 19
Other:
- note added: "G. Drive pass-through and DF0/DF1 swap"
- title: FluxDrive v1 rev A -> FluxDrive v1 rev B
- moved on the sheet: C1, C2, C3, C4, C5, C6, R1, R10, R11, R12, R13, R14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

Commit message: Rev B outputs: gated by SEL_FD_N, /CHNG and /INDEX from a west-end buffer
Parts:
- added C23: 1uF, Capacitor_SMD:C_0402_1005Metric, symbol Device:C
- added C24, C25: 10pF, Capacitor_SMD:C_0603_1608Metric, symbol Device:C
- added U10, U11: 74LVC32A, Package_SO:TSSOP-14_4.4x5mm_P0.65mm, symbol 74xx:74LS32
- added U17: SN74LVC2G07, Package_TO_SOT_SMD:SOT-23-6, symbol 74xGxx:74LVC2G07
- C10: value 47uF -> 100nF; footprint Capacitor_SMD:C_1206_3216Metric -> Capacitor_SMD:C_0402_1005Metric; LCSC C96123 -> C1525
- C11: value 47uF -> 1uF; footprint Capacitor_SMD:C_1206_3216Metric -> Capacitor_SMD:C_0402_1005Metric; LCSC C96123 -> C52923
- C12: value 100nF -> 22nF; LCSC C1525 -> C1532
- C13: value 10uF -> 47uF; footprint Capacitor_SMD:C_0603_1608Metric -> Capacitor_SMD:C_1206_3216Metric; LCSC C19702 -> C96123
- C14: value 100nF -> 47uF; footprint Capacitor_SMD:C_0402_1005Metric -> Capacitor_SMD:C_1206_3216Metric; LCSC C1525 -> C96123
- C15: value 4.7uF -> 100nF; footprint Capacitor_SMD:C_0603_1608Metric -> Capacitor_SMD:C_0402_1005Metric; LCSC (none) -> C1525; now fitted; now in the parts list
- C16: value 15pF -> 10uF; LCSC (none) -> C19702; now fitted; now in the parts list
- C17: value 22uF -> 100nF; footprint Capacitor_SMD:C_0805_2012Metric -> Capacitor_SMD:C_0402_1005Metric; LCSC C45783 -> C1525
- C18: value 22uF -> 4.7uF; footprint Capacitor_SMD:C_0805_2012Metric -> Capacitor_SMD:C_0603_1608Metric; LCSC C45783 -> (none); now not fitted; now left out of the parts list
- C19: value 100nF -> 15pF; footprint Capacitor_SMD:C_0402_1005Metric -> Capacitor_SMD:C_0603_1608Metric; LCSC C1525 -> (none); now not fitted; now left out of the parts list
- C20: value 1uF -> 22uF; footprint Capacitor_SMD:C_0402_1005Metric -> Capacitor_SMD:C_0805_2012Metric; LCSC C52923 -> C45783
- C21: value 10pF -> 22uF; footprint Capacitor_SMD:C_0603_1608Metric -> Capacitor_SMD:C_0805_2012Metric; LCSC (none) -> C45783; now fitted; now in the parts list
- C22: value 10pF -> 100nF; footprint Capacitor_SMD:C_0603_1608Metric -> Capacitor_SMD:C_0402_1005Metric; LCSC (none) -> C1525; now fitted; now in the parts list
- C8: value 1uF -> 100nF; LCSC C52923 -> C1525
- C9: value 22nF -> 100nF; LCSC C1532 -> C1525
Connections:
- net +3V3: now also C10.1, C20.1, C21.1, C22.1, C8.1, C9.1, U4.11, U4.9, U10.14 (VCC), U11.14 (VCC), U17.5 (VCC); no longer C16.1, C17.1, C18.1
- net +5V_A: now also C13.1, C14.1, C15.1; no longer C10.1, C11.1, C12.1
- net +5V_IN: now also C11.1; no longer C8.1
- net BUCK_FB: now also C19.2; no longer C16.2
- net CHNG_D: now also U17.6; no longer U4.10
- net CHNG_N: now also U11.1; no longer U4.11
- net DKRD_N: now also U10.1; no longer U4.3
- net EFUSE_DVDT: now also C12.1; no longer C9.1
- net ESP_EN: now also C23.1; no longer C20.1
- net GND: now also C16.2, C23.2, C24.2, C25.2, U10.7 (GND), U11.12, U11.13, U11.7 (GND), U17.2 (GND); no longer C19.2
- net INDEX_D: now also R45.1, U17.4; no longer R37.1, U4.8
- net INDEX_N: now also R44.1, U11.4; no longer R36.1, U4.9
- net RDY_D: now also R41.1; no longer R45.1
- net RDY_N: now also R40.1, U10.12; no longer R44.1, U4.5
- net SEL0: now also U11.9
- net SEL1: now also U11.10
- net SEL_FD_N: now also U10.10, U10.13, U10.2, U10.5, U11.2, U11.5
- net TRK0_D: now also R37.1; no longer R39.1
- net TRK0_N: now also R36.1, U10.4; no longer R38.1, U4.13
- net USB_DN: now also C25.1; no longer C22.1
- net USB_DP: now also C24.1; no longer C21.1
- net V5SYS: now also C16.1, C17.1; no longer C13.1, C14.1
- net V5SYS_DAMP: now also C18.1; no longer C15.1
- net WPROT_D: now also R39.1; no longer R41.1
- net WPROT_N: now also R38.1, U10.9; no longer R40.1, U4.1
- net _INDEX: now also R45.2; no longer R37.2
- net _RDY: now also R41.2; no longer R45.2
- net _TRK0: now also R37.2; no longer R39.2
- net _WPROT: now also R39.2; no longer R41.2
- new net BUSY: U11.8
- new net CHNG_G: U11.3, U17.1
- new net DKRD_G: U10.3, U4.3
- new net INDEX_G: U11.6, U17.3
- new net RDY_G: U10.11, U4.5
- new net TRK0_G: U10.6, U4.13
- new net WPROT_G: U10.8, U4.1
- no-connect marks 19 -> 22
Other:
- moved on the sheet: C10, C11, C12, C13, C14, C17, C20, C7, C8, C9, D1, D2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

Commit message: Rev B mode latch, select and clock gates, switch pads, J5 as a 4-pin header
Parts:
- added C26, C27, C28, C29, C32, C33: 100nF, Capacitor_SMD:C_0402_1005Metric, symbol Device:C
- added C30, C31: 1uF, Capacitor_SMD:C_0402_1005Metric, symbol Device:C
- added D5, D6: 1N4148W, Diode_SMD:D_SOD-123, symbol Device:D
- added J7: DF0 switch, Connector_PinHeader_2.54mm:PinHeader_1x03_P2.54mm_Vertical, symbol Connector_Generic:Conn_01x03
- added JP5: DF0 at power-on, Jumper:SolderJumper-3_P1.3mm_Bridged12_RoundedPad1.0x1.5mm, symbol Jumper:SolderJumper_3_Bridged12
- added JP6: REAL clear, Jumper:SolderJumper-2_P1.3mm_Open_RoundedPad1.0x1.5mm, symbol Jumper:SolderJumper_2_Open
- added JP7: REAL preset, Jumper:SolderJumper-2_P1.3mm_Open_RoundedPad1.0x1.5mm, symbol Jumper:SolderJumper_2_Open
- added R63, R64, R65, R66, R71, R72: 10K, Resistor_SMD:R_0402_1005Metric, symbol Device:R
- added R67, R68: 100K, Resistor_SMD:R_0402_1005Metric, symbol Device:R
- added R69, R70, R73, R74: 1K, Resistor_SMD:R_0402_1005Metric, symbol Device:R
- added U12, U13, U16: 74LVC1G157, Package_TO_SOT_SMD:SOT-363_SC-70-6, symbol FluxDrive:74LVC1G157
- added U8: 74LVC74A, Package_SO:TSSOP-14_4.4x5mm_P0.65mm, symbol 74xx:74LS74
- J5: value Spare GPIO -> Spare / OLED; footprint Connector_PinHeader_2.54mm:PinHeader_1x06_P2.54mm_Vertical -> Connector_PinHeader_2.54mm:PinHeader_1x04_P2.54mm_Vertical; symbol Connector_Generic:Conn_01x06 -> Connector_Generic:Conn_01x04
Connections:
- net +3V3: now also J5.2 (Pin_2), C26.1, C27.1, C28.1, C29.1, D5.1 (K), D6.1 (K), JP7.2 (B), R63.2, R64.2, R65.2, R66.2, U12.5 (VCC), U13.5 (VCC), U16.5 (VCC), U8.14 (VCC); no longer J5.5 (Pin_5)
- net BUSY: now also U16.6 (S)
- net GND: now also J5.1 (Pin_1), C26.2, C27.2, C28.2, C29.2, C30.2, C31.2, C32.2, C33.2, J7.2 (Pin_2), JP6.2 (B), R71.2, R72.2, U12.2 (GND), U12.3 (I0), U13.2 (GND), U16.1 (I1), U16.2 (GND), U8.7 (GND); no longer J5.6 (Pin_6)
- net SEL0: now also U13.1 (I1)
- net SEL1: now also U12.1 (I1)
- net SEL_FD: now also U13.4 (Y)
- net GPIO18: now reaches U1.11 (IO18)
- net GPIO18: now also J5.3 (Pin_3)
- net DF1_STATE: now reaches U1.12 (IO8)
- net DF1_STATE: now also R70.2
- net GPIO3: now reaches U1.15 (IO3)
- net GPIO3: now also J5.4 (Pin_4)
- net RST_REQ: now reaches U1.18 (IO10)
- net DF0_STATE: now reaches U1.20 (IO12)
- net DF0_STATE: now also R69.2
- net RST_ACT_IO: now reaches U1.4 (IO4)
- net GPIO13 renamed DF1_REQ
- net DF1_REQ: now also R68.2, U8.12 (D); no longer J5.1 (Pin_1)
- net GPIO14 renamed CHNG_REQ
- net CHNG_REQ: now also R72.1; no longer J5.2 (Pin_2)
- net GPIO47 renamed MODE_CLK_REQ
- net MODE_CLK_REQ: now also R71.1, U16.3 (I0); no longer J5.3 (Pin_3)
- net GPIO48 renamed DF0_REQ
- net DF0_REQ: now also R67.2, U8.2 (D); no longer J5.4 (Pin_4)
- new net CLR_A: JP5.1 (A), JP6.1 (A), R63.1, R74.2, U8.1 (~{R})
- new net CLR_B: C30.1, D5.2 (A), R65.1, U8.13 (~{R})
- new net DF0_FD: R67.1, R69.1, U13.6 (S), U8.5 (Q)
- new net DF1_EN: R68.1, R70.1, U12.6 (S), U8.9 (Q)
- new net J7_FD: C32.1, J7.1 (Pin_1), R73.1
- new net J7_REAL: C33.1, J7.3 (Pin_3), R74.1
- new net MODE_CLK: U16.4 (Y), U8.11 (C), U8.3 (C)
- new net POR_A: C31.1, D6.2 (A), JP5.2 (C)
- new net PRE_A: JP5.3 (B), JP7.1 (A), R64.1, R73.2, U8.4 (~{S})
- new net PRE_B: R66.1, U8.10 (~{S})
- new net SEL1_EN: U12.4 (Y), U13.3 (I0)
- no-connect marks 22 -> 18
Other:
- moved on the sheet: C21, C22, C23, R54, R55, SW1, SW2, U1

Commit message: Rev B J6 pass-through, real-drive drivers, bypass and mode-4 jumpers, virtual disk change
Parts:
- added C34, C35, C36, C37: 100nF, Capacitor_SMD:C_0402_1005Metric, symbol Device:C
- added J6: Original drive, Connector_IDC:IDC-Header_2x17_P2.54mm_Vertical, symbol Connector_Generic:Conn_02x17_Odd_Even
- added JP1: bypass SEL, Jumper:SolderJumper-3_P1.3mm_Bridged12_RoundedPad1.0x1.5mm, symbol Jumper:SolderJumper_3_Bridged12
- added JP2: bypass MTR, Jumper:SolderJumper-3_P1.3mm_Bridged12_RoundedPad1.0x1.5mm, symbol Jumper:SolderJumper_3_Bridged12
- added JP3: mode 4 SEL, Jumper:SolderJumper-3_P1.3mm_Bridged12_RoundedPad1.0x1.5mm, symbol Jumper:SolderJumper_3_Bridged12
- added JP4: mode 4 MTR, Jumper:SolderJumper-3_P1.3mm_Bridged12_RoundedPad1.0x1.5mm, symbol Jumper:SolderJumper_3_Bridged12
- added R75, R76: 4K7, Resistor_SMD:R_0402_1005Metric, symbol Device:R
- added R77, R78, R79: 10K, Resistor_SMD:R_0402_1005Metric, symbol Device:R
- added R80: 33, Resistor_SMD:R_0402_1005Metric, symbol Device:R
- added U14, U15: 74LVC1G157, Package_TO_SOT_SMD:SOT-363_SC-70-6, symbol FluxDrive:74LVC1G157
- added U18: SN74LVC2G06, Package_TO_SOT_SMD:SOT-23-6, symbol 74xGxx:74LVC2G06
- added U20: SN74LVC1G38, Package_TO_SOT_SMD:SOT-23-5, symbol 74xGxx:74LVC1G38
Connections:
- net +3V3: now also C34.1, C35.1, C36.1, C37.1, U14.5 (VCC), U15.5 (VCC), U18.5 (VCC), U20.5 (VCC)
- net +5V_A: now also R75.2, R76.2, R77.2, R78.2, R79.2
- net CHNG_REQ: now also U20.1
- net DF0_FD: now also U14.6 (S), U15.6 (S)
- net GND: now also C34.2, C35.2, C36.2, C37.2, J6.1 (Pin_1), J6.11 (Pin_11), J6.13 (Pin_13), J6.15 (Pin_15), J6.17 (Pin_17), J6.19 (Pin_19), J6.21 (Pin_21), J6.23 (Pin_23), J6.25 (Pin_25), J6.27 (Pin_27), J6.29 (Pin_29), J6.31 (Pin_31), J6.33 (Pin_33), J6.5 (Pin_5), J6.7 (Pin_7), J6.9 (Pin_9), JP3.1 (A), JP4.1 (A), U14.2 (GND), U15.2 (GND), U18.2 (GND), U20.3 (GND)
- net M4_MTR_Q: now also JP4.3 (B)
- net MTR0: now also U15.3 (I0)
- net SEL0: now also U14.3 (I0), U20.2
- net _CHNG: now also J6.2 (Pin_2), R80.2
- net _DIR: now also J6.18 (Pin_18)
- net _DKRD: now also J6.30 (Pin_30)
- net _DKWD: now also J6.22 (Pin_22)
- net _DKWE: now also J6.24 (Pin_24)
- net _INDEX: now also J6.8 (Pin_8)
- net _MTR0: now also JP2.3 (B)
- net _RDY: now also J6.34 (Pin_34)
- net _SEL0: now also JP1.3 (B)
- net _SIDE: now also J6.32 (Pin_32)
- net _STEP: now also J6.20 (Pin_20)
- net _TRK0: now also J6.26 (Pin_26)
- net _WPROT: now also J6.28 (Pin_28)
- new net J6_MTR: J6.16 (Pin_16), J6.4 (Pin_4), JP2.2 (C)
- new net J6_MTR_D: JP2.1 (A), R76.1, U18.4
- new net J6_PIN12: J6.12 (Pin_12), R78.1
- new net J6_PIN14: J6.14 (Pin_14), R79.1
- new net J6_PIN6: J6.6 (Pin_6), R77.1
- new net J6_SEL: J6.10 (Pin_10), JP1.2 (C)
- new net J6_SEL_D: JP1.1 (A), R75.1, U18.6
- new net M4_MTR: JP4.2 (C), U15.1 (I1)
- new net M4_SEL: JP3.2 (C), U14.1 (I1)
- new net M4_SEL_Q: JP3.3 (B)
- new net REAL_MTR: U15.4 (Y), U18.3
- new net REAL_SEL: U14.4 (Y), U18.1
- new net VCHNG_D: R80.1, U20.4
- no-connect marks 18 -> 19
