File: FluxDrive.kicad_sch (KiCad schematic)
At the start: 179 parts, among them J1 Amiga floppy 34, J2 Floppy power, J3 USB-C, J4 UART / recovery, J5 Spare / OLED, J6 Original drive, J7 DF0 switch, SW1 BOOT, SW2 RESET, U1 ESP32-S3-WROOM-1-N16R8, U10 74LVC32A, U11 74LVC32A, U12 74LVC1G157, U13 74LVC1G157, U14 74LVC1G157, U15 74LVC1G157, U16 74LVC1G157, U17 SN74LVC2G07, U18 SN74LVC2G06, U2 74LVC14A, U20 SN74LVC1G38, U3 74LVC14A, U4 74LVC07A, U5 TPS259531, U6 TLV62569DBVR, U7 USBLC6-2SC6, U8 74LVC74A

Commit message: Rev B mode 4 as unfitted pads, the optional reset wire
Parts:
- added C38: 100nF, Capacitor_SMD:C_0402_1005Metric, symbol Device:C
- added C39, C40, C41: 100nF, Capacitor_SMD:C_0603_1608Metric, symbol Device:C
- added J10: MTRX wire, TestPoint:TestPoint_THTPad_D1.5mm_Drill0.7mm, symbol Connector:TestPoint
- added J9: RST wire, TestPoint:TestPoint_THTPad_D1.5mm_Drill0.7mm, symbol Connector:TestPoint
- added R81: 10K, Resistor_SMD:R_0402_1005Metric, symbol Device:R
- added R82: 1K, Resistor_SMD:R_0402_1005Metric, symbol Device:R
- added R83: 33, Resistor_SMD:R_0603_1608Metric, symbol Device:R
- added U19: SN74LVC1G06, Package_TO_SOT_SMD:SOT-23-5, symbol 74xGxx:74LVC1G06
- added U21: 74LVC1G157, Package_TO_SOT_SMD:SOT-363_SC-70-6, symbol FluxDrive:74LVC1G157
- added U22: SN74LVC1G175, Package_TO_SOT_SMD:SOT-23-6, symbol 74xGxx:74LVC1G175
- added U23: SN74LVC1G38, Package_TO_SOT_SMD:SOT-23-5, symbol 74xGxx:74LVC1G38
Connections:
- net +3V3: now also C38.1, C39.1, C40.1, C41.1, U19.5 (VCC), U21.5 (VCC), U22.5 (VCC), U23.5 (VCC)
- net DF0_FD: now also U21.6 (S)
- net DF1_EN: now also U22.6 (~{CLR})
- net GND: now also C38.2, C39.2, C40.2, C41.2, R81.2, U19.3 (GND), U21.2 (GND), U21.3 (I0), U22.2 (GND), U23.3 (GND)
- net KBRESET: now also J9.1, U19.4
- net M4_MOTOR: now also U22.3 (D)
- net M4_MTR_N: now also U23.2
- net M4_MTR_Q: now also U22.4 (Q)
- net M4_SEL_Q: now also U21.4 (Y), U23.1
- net MTRX: now also J10.1
- net RST_ACT: now also R82.1
- net RST_ACT_IO: now also R82.2
- net RST_REQ: now also R81.1, U19.2
- net SEL1: now also U22.1 (C)
- net SEL1_EN: now also U21.1 (I1)
- net _RDY: now also R83.2
- new net ID_D: R83.1, U23.4
