File: FluxDrive.kicad_sch (KiCad schematic)
At the start: 192 parts, among them J1 Amiga floppy 34, J10 MTRX wire, J2 Floppy power, J3 USB-C, J4 UART / recovery, J5 Spare / OLED, J6 Original drive, J7 DF0 switch, J9 RST wire, SW1 BOOT, SW2 RESET, U1 ESP32-S3-WROOM-1-N16R8, U10 74LVC32A, U11 74LVC32A, U12 74LVC1G157, U13 74LVC1G157, U14 74LVC1G157, U15 74LVC1G157, U16 74LVC1G157, U17 SN74LVC2G07, U18 SN74LVC2G06, U19 SN74LVC1G06, U2 74LVC14A, U20 SN74LVC1G38, U21 74LVC1G157, U22 SN74LVC1G175, U23 SN74LVC1G38, U3 74LVC14A, U4 74LVC07A, U5 TPS259531, U6 TLV62569DBVR, U7 USBLC6-2SC6, U8 74LVC74A

Commit message: Rev B drive power behind its own eFuse, test pads; the steering logic proven on the netlist
Parts:
- added C42: 100nF, Capacitor_SMD:C_0402_1005Metric, symbol Device:C
- added C43, C44, C45: 100nF, Capacitor_SMD:C_0603_1608Metric, symbol Device:C
- added J8: Drive power, FluxDrive:171825-4, symbol FluxDrive:171825-4
- added R84: 33, Resistor_SMD:R_0603_1608Metric, symbol Device:R
- added TP17: SEL_FD, TestPoint:TestPoint_Pad_D1.0mm, symbol Connector:TestPoint
- added TP18: REAL_SEL, TestPoint:TestPoint_Pad_D1.0mm, symbol Connector:TestPoint
- added TP19: REAL_MTR, TestPoint:TestPoint_Pad_D1.0mm, symbol Connector:TestPoint
- added TP20: DF0_STATE, TestPoint:TestPoint_Pad_D1.0mm, symbol Connector:TestPoint
- added TP21: DF1_STATE, TestPoint:TestPoint_Pad_D1.0mm, symbol Connector:TestPoint
- added TP22: MODE_CLK, TestPoint:TestPoint_Pad_D1.0mm, symbol Connector:TestPoint
- added U9: TPS259531, Package_SON:Texas_DSG0008A_WSON-8-1EP_2x2mm_P0.5mm_EP0.9x1.6mm, symbol FluxDrive:TPS259531
- C13: value 47uF -> 1uF; footprint Capacitor_SMD:C_1206_3216Metric -> Capacitor_SMD:C_0402_1005Metric; LCSC C96123 -> C52923
- C14: value 47uF -> 22nF; footprint Capacitor_SMD:C_1206_3216Metric -> Capacitor_SMD:C_0402_1005Metric; LCSC C96123 -> C1532
- C15: value 100nF -> 22uF; footprint Capacitor_SMD:C_0402_1005Metric -> Capacitor_SMD:C_0805_2012Metric; LCSC C1525 -> C45783
- C16: value 10uF -> 100nF; footprint Capacitor_SMD:C_0603_1608Metric -> Capacitor_SMD:C_0402_1005Metric; LCSC C19702 -> C1525
- C17: value 100nF -> 47uF; footprint Capacitor_SMD:C_0402_1005Metric -> Capacitor_SMD:C_1206_3216Metric; LCSC C1525 -> C96123
- C18: value 4.7uF -> 47uF; footprint Capacitor_SMD:C_0603_1608Metric -> Capacitor_SMD:C_1206_3216Metric; LCSC (none) -> C96123; now fitted; now in the parts list
- C19: value 15pF -> 100nF; footprint Capacitor_SMD:C_0603_1608Metric -> Capacitor_SMD:C_0402_1005Metric; LCSC (none) -> C1525; now fitted; now in the parts list
- C20: value 22uF -> 10uF; footprint Capacitor_SMD:C_0805_2012Metric -> Capacitor_SMD:C_0603_1608Metric; LCSC C45783 -> C19702
- C21: value 22uF -> 100nF; footprint Capacitor_SMD:C_0805_2012Metric -> Capacitor_SMD:C_0402_1005Metric; LCSC C45783 -> C1525
- C22: value 100nF -> 4.7uF; footprint Capacitor_SMD:C_0402_1005Metric -> Capacitor_SMD:C_0603_1608Metric; LCSC C1525 -> (none); now not fitted; now left out of the parts list
- C23: value 1uF -> 15pF; footprint Capacitor_SMD:C_0402_1005Metric -> Capacitor_SMD:C_0603_1608Metric; LCSC C52923 -> (none); now not fitted; now left out of the parts list
- C24, C25: value 10pF -> 22uF; footprint Capacitor_SMD:C_0603_1608Metric -> Capacitor_SMD:C_0805_2012Metric; LCSC (none) -> C45783; now fitted; now in the parts list
- C27, C34, C35: value 100nF -> 1uF; LCSC C1525 -> C52923
- C28, C29: value 100nF -> 10pF; footprint Capacitor_SMD:C_0402_1005Metric -> Capacitor_SMD:C_0603_1608Metric; LCSC C1525 -> (none); now not fitted; now left out of the parts list
- C30, C31: value 1uF -> 100nF; LCSC C52923 -> C1525
- C39, C40, C41: footprint Capacitor_SMD:C_0603_1608Metric -> Capacitor_SMD:C_0402_1005Metric; LCSC (none) -> C1525; now fitted; now in the parts list
- R49: value 1R -> 1K37; footprint Resistor_SMD:R_0603_1608Metric -> Resistor_SMD:R_0402_1005Metric; LCSC (none) -> C423239; now fitted; now in the parts list
- R50: value 100K -> 1R; footprint Resistor_SMD:R_0402_1005Metric -> Resistor_SMD:R_0603_1608Metric; LCSC C25741 -> (none); now not fitted; now left out of the parts list
- R51: value 22K -> 100K; LCSC C25768 -> C25741
- R52: value 1K -> 22K; LCSC C11702 -> C25768
- R53: value 1K5 -> 1K; LCSC C25867 -> C11702
- R54: value 10K -> 1K5; LCSC C25744 -> C25867
- R56: value 5K1 -> 10K; LCSC C25905 -> C25744
- R58: value 10K -> 5K1; LCSC C25744 -> C25905
- R59: value 22 -> 10K; LCSC C25092 -> C25744
- R61: value 470 -> 22; LCSC C25117 -> C25092
- R62: value 1K -> 470; LCSC C11702 -> C25117
- R63, R71: value 10K -> 1K; LCSC C25744 -> C11702
- R67: value 100K -> 10K; LCSC C25741 -> C25744
- R69: value 1K -> 100K; LCSC C11702 -> C25741
- R73, R82: value 1K -> 10K; LCSC C11702 -> C25744
- R75: value 4K7 -> 1K; LCSC C25900 -> C11702
- R77: value 10K -> 4K7; LCSC C25744 -> C25900
- R80: value 33 -> 10K; LCSC C25105 -> C25744
- R81: value 10K -> 33; LCSC C25744 -> C25105
- R83: value 33 -> 1K; footprint Resistor_SMD:R_0603_1608Metric -> Resistor_SMD:R_0402_1005Metric; LCSC (none) -> C11702; now fitted; now in the parts list
Connections:
- net +3V3: now also C23.1, C24.1, C25.1, C30.1, C31.1, C32.1, C33.1, R51.1, R56.1, R67.2, C42.1, C43.1, C44.1, C45.1; no longer C19.1, C20.1, C21.1, C22.1, C27.1, C28.1, C29.1, C34.1, C35.1, C36.1, C37.1, R50.1, R54.1, R63.2
- net +5V_A: now also C17.1, C18.1, C19.1, R53.1, R80.2; no longer C13.1, C14.1, C15.1, R52.1, R75.2
- net +5V_IN: now also C13.1, U9.3 (IN), U9.4 (IN)
- net AMIGA_PWR: now also R53.2, R54.1; no longer R52.2, R53.1
- net BOOT: now also R56.2; no longer R55.2
- net BUCK_FB: now also C23.2, R51.2, R52.1; no longer C19.2, R50.2, R51.1
- net CHNG_REQ: now also R73.1; no longer R72.1
- net CLR_A: now also R64.1, R75.2; no longer R63.1, R74.2
- net CLR_B: now also C34.1, R66.1; no longer C30.1, R65.1
- net DF0_FD: now also R68.1, R70.1; no longer R67.1, R69.1
- net DF0_REQ: now also R68.2; no longer R67.2
- net DF0_STATE: now also R70.2, TP20.1; no longer R69.2
- net DF1_EN: now also R69.1, R71.1; no longer R68.1, R70.1
- net DF1_REQ: now also R69.2; no longer R68.2
- net DF1_STATE: now also R71.2, TP21.1; no longer R70.2
- net EFUSE_EN: now also U9.2 (EN/UVLO)
- net ESP_EN: now also C27.1, R55.2; no longer C23.1, R54.2
- net ESP_TXD0: now also R62.1; no longer R61.1
- net GND: now also C19.2, R49.2, R52.2, R54.2, R59.2, R73.2, R82.2, C42.2, C43.2, C44.2, C45.2, J8.2 (GND), J8.3 (GND), U9.8 (GND), U9.9 (PAD); no longer C23.2, R51.2, R53.2, R56.2, R71.2, R81.2
- net ID_D: now also R84.1; no longer R83.1
- net J6_MTR_D: now also R77.1; no longer R76.1
- net J6_PIN12: now also R79.1; no longer R78.1
- net J6_PIN14: now also R80.1; no longer R79.1
- net J6_PIN6: now also R78.1; no longer R77.1
- net J6_SEL_D: now also R76.1; no longer R75.1
- net J7_FD: now also C36.1, R74.1; no longer C32.1, R73.1
- net J7_REAL: now also C37.1, R75.1; no longer C33.1, R74.1
- net LED: now also R63.1; no longer R62.1
- net LED_A: now also R63.2; no longer R62.2
- net MODE_CLK: now also TP22.1
- net MODE_CLK_REQ: now also R72.1; no longer R71.1
- net POR_A: now also C35.1; no longer C31.1
- net PRE_A: now also R65.1, R74.2; no longer R64.1, R73.2
- net PRE_B: now also R67.1; no longer R66.1
- net REAL_MTR: now also TP19.1
- net REAL_SEL: now also TP18.1
- net RST_ACT: now also R83.1; no longer R82.1
- net RST_ACT_IO: now also R83.2; no longer R82.2
- net RST_REQ: now also R82.1; no longer R81.1
- net SEL_FD: now also TP17.1
- net UART_TX: now also R62.2; no longer R61.2
- net USB_CC1: now also R57.1; no longer R56.1
- net USB_CC2: now also R58.1; no longer R57.1
- net USB_DN: now also C29.1, R61.2; no longer C25.1, R60.2
- net USB_DN_C: now also R61.1; no longer R60.1
- net USB_DP: now also C28.1, R60.2; no longer C24.1, R59.2
- net USB_DP_C: now also R60.1; no longer R59.1
- net V5SYS: now also C20.1, C21.1, R50.1; no longer C16.1, C17.1, R49.1
- net V5SYS_DAMP: now also C22.1, R50.2; no longer C18.1, R49.2
- net VBUS: now also R59.1; no longer R58.1
- net VCHNG_D: now also R81.1; no longer R80.1
- net _CHNG: now also R81.2; no longer R80.2
- net _RDY: now also R84.2; no longer R83.2
- net +12V: now reaches J2.4 (12V)
- net +12V: now also J8.4 (12V)
- new net +5V_DRIVE: C15.1, C16.1, J8.1 (5V), U9.5 (OUT)
- new net DRV_DVDT: C14.1, U9.1 (dVdt)
- new net DRV_ILM: R49.1, U9.7 (ILM)
Other:
- moved on the sheet: C13, C14, C15, C16, C17, C20, C21, C26, C27, C30, C31, C32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

Commit message: Rev B schematic review and fixes
Fixes from the four specialist reviews of 329c6e9, each with a test:
- U4 is the Diodes 74LVC07AS14-13 (C176925); C6049 has no stock (RPCB-1).
- R85: 100 kOhm from M4_SEL_Q to GND, so a partly fitted mode-4 kit cannot
  leave the real drive's select floating (RBUS-1).
- Test pads TP20/TP21 on DF0_FD/DF1_EN, the latch side (RESP-1).
- The mode-4 DNP parts keep their LCSC numbers (RPCB-6).
- Evaluator: a live gate with a floating input gives its output no level
  (RBUS-8).
- sch_gen raises on a repeated ref (RCODE-1).
- New tests: mode-4 latch sequence and kit values, reset wire input, strap
  pins, partial mode-4 fit, BOM exclusions as a written-out set, test pads
  by equality, C13 and the drive eFuse's 1.30 A minimum limit (RBUS-2/3/4/7,
  RCODE-4/7, RPWR-1/6).
- design.py docstring and dead entries tidied (RCODE-5/6).

Schematic and PDF regenerated: ERC 0 errors, 27 footprint_filter. Suite 333
passed, 48 skipped; build/revb/mutate.py still catches all 6 mutants.
Parts:
- added R85: 100K, Resistor_SMD:R_0402_1005Metric, symbol Device:R
- TP20: value DF0_STATE -> DF0_FD
- TP21: value DF1_STATE -> DF1_EN
- U21: LCSC (none) -> C135822
- U23: LCSC (none) -> C2867613
- U4: LCSC C6049 -> C176925
Connections:
- net DF0_FD: now also TP20.1
- net DF0_STATE: no longer TP20.1
- net DF1_EN: now also TP21.1
- net DF1_STATE: no longer TP21.1
- net GND: now also R85.2
- net M4_SEL_Q: now also R85.1
Changed lines of the file:
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@@
 			)
 		)
-		(property "LCSC" "C6049"
+		(property "LCSC" "C176925"
 			(at 429.26 181.61 0)
 			(hide yes)
@@
 			)
 		)
-		(property "LCSC" "C6049"
+		(property "LCSC" "C176925"
 			(at 472.44 181.61 0)
 			(hide yes)
@@
 			)
 		)
-		(property "LCSC" "C6049"
+		(property "LCSC" "C176925"
 			(at 511.81 181.61 0)
 			(hide yes)
@@
 			)
 		)
-		(property "LCSC" "C6049"
+		(property "LCSC" "C176925"
 			(at 551.18 181.61 0)
 			(hide yes)
@@
 			)
 		)
-		(property "LCSC" "C6049"
+		(property "LCSC" "C176925"
 			(at 584.2 181.61 0)
 			(hide yes)
@@
 			)
 		)
-		(property "LCSC" "C6049"
+		(property "LCSC" "C176925"
 			(at 619.76 181.61 0)
 			(hide yes)
@@
 			)
 		)
-		(property "LCSC" "C6049"
+		(property "LCSC" "C176925"
 			(at 645.16 200.66 0)
 			(hide yes)
@@
 			)
 		)
-		(property "Value" "DF0_STATE"
+		(property "Value" "DF0_FD"
 			(at 360.68 588.01 0)
 			(effects
@@
 		)
 	)
-	(label "DF0_STATE"
+	(label "DF0_FD"
 		(at 360.68 582.93 270)
 		(effects
@@
 			)
 		)
-		(property "Value" "DF1_STATE"
+		(property "Value" "DF1_EN"
 			(at 370.84 588.01 0)
 			(effects
@@
 		)
 	)
-	(label "DF1_STATE"
+	(label "DF1_EN"
 		(at 370.84 582.93 270)
 		(effects
@@
 			)
 		)
+		(property "LCSC" "C135822"
+			(at 918.21 712.47 0)
+			(hide yes)
+			(effects
+				(font
+					(size 1.27 1.27)
+				)
+			)
+		)
 		(pin "1"
 		)
@@
 			)
 		)
+		(property "LCSC" "C2867613"
+			(at 1084.58 715.01 0)
+			(hide yes)
+			(effects
+				(font
+					(size 1.27 1.27)
+				)
+			)
+		)
 		(pin "1"
 		)
@@
 	)
 	(symbol
+		(lib_id "Device:R")
+		(at 36.83 764.54 90)
+		(unit 1)
+		(body_style 1)
+		(exclude_from_sim no)
+		(in_bom yes)
+		(on_board yes)
+		(in_pos_files yes)
+		(dnp no)
+		(property "Reference" "R85"
+			(at 36.83 759.46 90)
+			(effects
+				(font
+					(size 1.27 1.27)
+				)
+			)
+		)
+		(property "Value" "100K"
+			(at 36.83 769.62 90)
+			(effects
+				(font
+					(size 1.27 1.27)
+				)
+			)
+		)
+		(property "Footprint" "Resistor_SMD:R_0402_1005Metric"
+			(at 36.83 764.54 0)
+			(hide yes)
+			(effects
+				(font
+					(size 1.27 1.27)
+				)
+			)
+		)
+		(property "Datasheet" ""
+			(at 36.83 764.54 0)
+			(hide yes)
+			(effects
+				(font
+					(size 1.27 1.27)
+				)
+			)
+		)
+		(property "LCSC" "C25741"
+			(at 36.83 764.54 0)
+			(hide yes)
+			(effects
+				(font
+					(size 1.27 1.27)
+				)
+			)
+		)
+		(pin "1"
+		)
+		(pin "2"
+		)
+		(instances
+			(project "FluxDrive"
+				(path "/d01aa0ea-135a-52e5-ab1a-3ab06ba49a4e"
+					(reference "R85")
+					(unit 1)
+				)
+			)
+		)
+	)
+	(label "M4_SEL_Q"
+		(at 33.02 764.54 180)
+		(effects
+			(font
+				(size 1.27 1.27)
+			)
+			(justify right bottom)
+		)
+	)
+	(label "GND"
+		(at 40.64 764.54 0)
+		(effects
+			(font
+				(size 1.27 1.27)
+			)
+			(justify left bottom)
+		)
+	)
+	(symbol
 		(lib_id "power:PWR_FLAG")
-		(at 22.86 764.54 0)
+		(at 55.88 764.54 0)
 		(unit 1)
 		(body_style 1)
@@
 		(dnp no)
 		(property "Reference" "#FLG01"
-			(at 22.86 759.46 0)
+			(at 55.88 759.46 0)
 			(effects
 				(font
@@
 		)
 		(property "Value" "PWR_FLAG"
-			(at 22.86 769.62 0)
+			(at 55.88 769.62 0)
 			(effects
 				(font
@@
 		)
 		(property "Footprint" ""
-			(at 22.86 764.54 0)
+			(at 55.88 764.54 0)
 			(hide yes)
 			(effects
@@
 		)
 		(property "Datasheet" ""
-			(at 22.86 764.54 0)
+			(at 55.88 764.54 0)
 			(hide yes)
 			(effects
@@
 	)
 	(label "GND"
-		(at 22.86 764.54 270)
+		(at 55.88 764.54 270)
 		(effects
 			(font
@@
 	(symbol
 		(lib_id "power:PWR_FLAG")
-		(at 33.02 764.54 0)
+		(at 66.04 764.54 0)
 		(unit 1)
 		(body_style 1)
@@
 		(dnp no)
 		(property "Reference" "#FLG02"
-			(at 33.02 759.46 0)
+			(at 66.04 759.46 0)
 			(effects
 				(font
@@
 		)
 		(property "Value" "PWR_FLAG"
-			(at 33.02 769.62 0)
+			(at 66.04 769.62 0)
 			(effects
 				(font
@@
 		)
 		(property "Footprint" ""
-			(at 33.02 764.54 0)
+			(at 66.04 764.54 0)
 			(hide yes)
 			(effects
@@
 		)
 		(property "Datasheet" ""
-			(at 33.02 764.54 0)
+			(at 66.04 764.54 0)
 			(hide yes)
 			(effects
@@
 	)
 	(label "+3V3"
-		(at 33.02 764.54 270)
+		(at 66.04 764.54 270)
 		(effects
 			(font
@@
 	(symbol
 		(lib_id "power:PWR_FLAG")
-		(at 43.18 764.54 0)
+		(at 76.2 764.54 0)
 		(unit 1)
 		(body_style 1)
@@
 		(dnp no)
 		(property "Reference" "#FLG03"
-			(at 43.18 759.46 0)
+			(at 76.2 759.46 0)
 			(effects
 				(font
@@
 		)
 		(property "Value" "PWR_FLAG"
-			(at 43.18 769.62 0)
+			(at 76.2 769.62 0)
 			(effects
 				(font
@@
 		)
 		(property "Footprint" ""
-			(at 43.18 764.54 0)
+			(at 76.2 764.54 0)
 			(hide yes)
 			(effects
@@
 		)
 		(property "Datasheet" ""
-			(at 43.18 764.54 0)
+			(at 76.2 764.54 0)
 			(hide yes)
 			(effects
@@
 	)
 	(label "+5V_IN"
-		(at 43.18 764.54 270)
+		(at 76.2 764.54 270)
 		(effects
 			(font
@@
 	(symbol
 		(lib_id "power:PWR_FLAG")
-		(at 53.34 764.54 0)
+		(at 86.36 764.54 0)
 		(unit 1)
 		(body_style 1)
@@
 		(dnp no)
 		(property "Reference" "#FLG04"
-			(at 53.34 759.46 0)
+			(at 86.36 759.46 0)
 			(effects
 				(font
@@
 		)
 		(property "Value" "PWR_FLAG"
-			(at 53.34 769.62 0)
+			(at 86.36 769.62 0)
 			(effects
 				(font
@@
 		)
 		(property "Footprint" ""
-			(at 53.34 764.54 0)
+			(at 86.36 764.54 0)
 			(hide yes)
 			(effects
@@
 		)
 		(property "Datasheet" ""
-			(at 53.34 764.54 0)
+			(at 86.36 764.54 0)
 			(hide yes)
 			(effects
@@
 	)
 	(label "V5SYS"
-		(at 53.34 764.54 270)
+		(at 86.36 764.54 270)
 		(effects
 			(font
@@
 	(symbol
 		(lib_id "power:PWR_FLAG")
-		(at 63.5 764.54 0)
+		(at 96.52 764.54 0)
 		(unit 1)
 		(body_style 1)
@@
 		(dnp no)
 		(property "Reference" "#FLG05"
-			(at 63.5 759.46 0)
+			(at 96.52 759.46 0)
 			(effects
 				(font
@@
 		)
 		(property "Value" "PWR_FLAG"
-			(at 63.5 769.62 0)
+			(at 96.52 769.62 0)
 			(effects
 				(font
@@
 		)
 		(property "Footprint" ""
-			(at 63.5 764.54 0)
+			(at 96.52 764.54 0)
 			(hide yes)
 			(effects
@@
 		)
 		(property "Datasheet" ""
-			(at 63.5 764.54 0)
+			(at 96.52 764.54 0)
 			(hide yes)
 			(effects
@@
 	)
 	(label "VBUS"
-		(at 63.5 764.54 270)
+		(at 96.52 764.54 270)
 		(effects
 			(font
